File: AgriESC.sch (KiCad schematic (older format))
At the start: 12 parts

Commit message: Added CAN, USB, hall sensors, servo
Parts:
- added C? (x6): 2u2, symbol Device:C
- added C?: 100n, symbol Device:C
- added D?: BLUE, symbol Device:LED_ALT
- added D?: GREEN, symbol Device:LED_ALT
- added D?: RED, symbol Device:LED_ALT
- added J?: USB_OTG, symbol Connector:USB_OTG
- added J?: HALL_ENC, symbol Connector_Generic:Conn_01x06
- added J?: CAN, symbol Connector_Generic:Conn_01x04
- added J?: SERVO, symbol Connector_Generic:Conn_01x03
- added R?: 1k, symbol Device:R
- added R? (x3): 220R, symbol Device:R
- added R?: 0R, symbol Device:R
- added R? (x2): 22R, symbol Device:R
- added R? (x3): 2k2, symbol Device:R
- added R?: 10k, symbol Device:R
- added SW?: SW_SPDT, symbol Switch:SW_SPDT
- added U?: TJA1051TK-3, Package_DFN_QFN:DFN-8-1EP_3x3mm_P0.65mm_EP1.55x2.4mm, symbol Interface_CAN_LIN:TJA1051TK-3
Connections:
- net labels added: +5V, CANH, CANL, CAN_RX, CAN_TX, RX, TX
- net labels removed: LED_GREEN, LED_RED
- wire segments 106 -> 198
- no-connect marks 7 -> 6
Other:
- note added: "Bypass"
- note added: "Optional"
- note removed: "CAN Bus"

Commit message: Started adding driver
Parts:
- added C?: 0.1u, symbol Device:C
- added C? (x2): C, symbol Device:C
- added J?: PH_A, symbol Connector_Generic:Conn_01x01
- added R?: 0.004R, symbol Device:R
- added R?: 59k, symbol Device:R
- added R?: 1k, symbol Device:R
- added R? (x2): R, symbol Device:R
- added U?: MAX9920, symbol AgriESC:MAX9920
- added U? (x2): FDMS7698, symbol AgriESC:FDMS7698
- added U?: DRV8303, symbol AgriESC:DRV8303
Connections:
- net labels added: C_A, GH_A, GL_A, SH_A, SL_A, SUPPLY
- wire segments 198 -> 244
Other:
- note added: "Gain set to 15"

Commit message: First draft of schematic complete
Parts:
- removed C? (x2): 2u2, symbol Device:C
- removed R?: 220R, symbol Device:R
- removed U?: TJA1051TK-3, Package_DFN_QFN:DFN-8-1EP_3x3mm_P0.65mm_EP1.55x2.4mm, symbol Interface_CAN_LIN:TJA1051TK-3
- added C1, C3, C4, C40, C41, C6, C7, C8, C9: 2u2, symbol Device:C
- added C11: 4u7_50V, symbol Device:C
- added C13, C14, C15: 220n, symbol Device:C
- added C16: 100n, symbol Device:C
- added C17: 10u, symbol Device:C
- added C28, C34: 0.1u, symbol Device:C
- added C30, C33, C35, C36: 4.7u_60V, symbol Device:C
- added C37, C38, C39: 4n7, symbol Device:C
- added C5: 22n, symbol Device:C
- added D4: D_Schottky_40V_1A, symbol Device:D_Schottky
- added J10: SWD, symbol Connector_Generic:Conn_01x05
- added J11: COMM, symbol Connector_Generic:Conn_01x08
- added J12: GPIO, symbol Connector_Generic:Conn_01x06
- added J6: PH_B, symbol Connector_Generic:Conn_01x01
- added J7: PH_C, symbol Connector_Generic:Conn_01x01
- added J8: SUPPLY, symbol Connector_Generic:Conn_01x01
- added J9: GND, symbol Connector_Generic:Conn_01x01
- added L1: 22u, symbol Device:L
- added R1, R3, R5, R7: 47k, symbol Device:R
- added R15: 220R, symbol Device:R
- added R2, R4, R6, R8: 5k6, symbol Device:R
- added R25, R33: 0.004R, symbol Device:R
- added R29, R34: 59k, symbol Device:R
- added R30, R35: 1k, symbol Device:R
- added R31, R32, R36, R37: 4R7, symbol Device:R
- added R38, R39, R40: 100R, symbol Device:R
- added R41: 100k, symbol Device:R
- added R42: 54k9, symbol Device:R
- added R43, R9: 10k, symbol Device:R
- added U10, U12, U13, U9: FDMS7698, symbol AgriESC:FDMS7698
- added U11, U8: MAX9920, symbol AgriESC:MAX9920
- added U14: MCP1700-3302E_SOT23, Package_TO_SOT_SMD:SOT-23, symbol Regulator_Linear:MCP1700-3302E_SOT23
- added U3: LMR16006YQ, Package_TO_SOT_SMD:SOT-23-6, symbol Regulator_Switching:LMR16006YQ
- added U4: TJA1051TK-3, Package_DFN_QFN:DFN-8-1EP_3x3mm_P0.65mm_EP1.55x2.4mm, symbol Interface_CAN_LIN:TJA1051TK-3
- C10, C12: renamed from C?; value C -> 4.7u_60V
- R13, R14: renamed from R?; value R -> 4R7
- R23: renamed from R?; value 10kNTC -> 10k_NTC
- gave numbers to parts that had none: 43
Connections:
- net labels added: CS, C_B, C_C, GH_B, GH_C, GL_B, GL_C, INH_A, INH_B, INH_C, INL_A, INL_B, INL_C, SCLK, SDI, SDO, SENS_A, SENS_B, SENS_C, SH_B, SH_C, SL_B, SL_C
- net labels removed: ADC_TEMP, RX, SENS_1, SENS_2, SENS_3, SPI3_CS, SPI3_MISO, SPI3_MOSI, SPI3_SCK, TX, VAA
- wire segments 244 -> 553
- no-connect marks 6 -> 10
Other:
- note added: "ADC_TEMP"
- note added: "From the design guide"
- note added: "Gives approx 3.2 V at 30 V input"
- note removed: "VAA?"

Commit message: Started allocating footprints
Parts:
- C1, C10, C11, C12, C13, C14, C15, C16, C17, C18, C19, C2, C20, C21, C22, C23, C24, C25, C26, C27, C28, C29, C3, C30, C31, C32, C33, C34, C35, C36, C37, C38, C39, C4, C40, C41, C5, C6, C7, C8, C9: footprint (none) -> Capacitor_SMD:C_0805_2012Metric_Pad1.15x1.40mm_HandSolder
- D1, D2, D3: footprint (none) -> LED_SMD:LED_0805_2012Metric_Pad1.15x1.40mm_HandSolder
- J10: footprint (none) -> Connector_PinHeader_2.54mm:PinHeader_1x05_P2.54mm_Vertical
- J11: footprint (none) -> Connector_PinHeader_2.54mm:PinHeader_1x08_P2.54mm_Vertical
- J12, J2: footprint (none) -> Connector_PinHeader_2.54mm:PinHeader_1x06_P2.54mm_Vertical
- J3: footprint (none) -> Connector_PinHeader_2.54mm:PinHeader_1x04_P2.54mm_Vertical
- J4: footprint (none) -> Connector_PinHeader_2.54mm:PinHeader_1x03_P2.54mm_Vertical
- J5: footprint (none) -> Connector_USB:USB_Micro-B_Amphenol_10103594-0001LF_Horizontal
- R1, R11, R12, R13, R14, R15, R16, R17, R18, R19, R2, R20, R21, R22, R24, R26, R27, R28, R29, R3, R30, R31, R32, R35, R36, R37, R38, R39, R4, R40, R41, R42, R43, R5, R6, R7, R8, R9: footprint (none) -> Resistor_SMD:R_0805_2012Metric_Pad1.15x1.40mm_HandSolder

Commit message: Added MAX9920 footprint to schematic
Parts:
- R10, R25, R33: footprint (none) -> Resistor_SMD:R_2512_6332Metric_Pad1.52x3.35mm_HandSolder
- R34: footprint (none) -> Resistor_SMD:R_0805_2012Metric_Pad1.15x1.40mm_HandSolder
- U1: footprint (none) -> AgriESC:MAX9920
Changed lines of the file:
@@
 F 0 "U1" H 1650 -1122 50  0000 C CNN
 F 1 "MAX9920" H 1650 -1213 50  0000 C CNN
-F 2 "" H 1650 -800 50  0001 C CNN
+F 2 "AgriESC:MAX9920" H 1650 -800 50  0001 C CNN
 F 3 "" H 1650 -800 50  0001 C CNN
 	1    1650 -750
@@
 F 0 "R10" V 1443 -1400 50  0000 C CNN
 F 1 "0.004R" V 1534 -1400 50  0000 C CNN
-F 2 "" V 1580 -1400 50  0001 C CNN
+F 2 "Resistor_SMD:R_2512_6332Metric_Pad1.52x3.35mm_HandSolder" V 1580 -1400 50  0001 C CNN
 F 3 "~" H 1650 -1400 50  0001 C CNN
 	1    1650 -1400
@@
 F 0 "R25" V 4743 -1400 50  0000 C CNN
 F 1 "0.004R" V 4834 -1400 50  0000 C CNN
-F 2 "" V 4880 -1400 50  0001 C CNN
+F 2 "Resistor_SMD:R_2512_6332Metric_Pad1.52x3.35mm_HandSolder" V 4880 -1400 50  0001 C CNN
 F 3 "~" H 4950 -1400 50  0001 C CNN
 	1    4950 -1400
@@
 F 0 "R33" V 7993 -1400 50  0000 C CNN
 F 1 "0.004R" V 8084 -1400 50  0000 C CNN
-F 2 "" V 8130 -1400 50  0001 C CNN
+F 2 "Resistor_SMD:R_2512_6332Metric_Pad1.52x3.35mm_HandSolder" V 8130 -1400 50  0001 C CNN
 F 3 "~" H 8200 -1400 50  0001 C CNN
 	1    8200 -1400
@@
 F 0 "R34" H 8770 -804 50  0000 L CNN
 F 1 "59k" H 8770 -895 50  0000 L CNN
-F 2 "" V 8630 -850 50  0001 C CNN
+F 2 "Resistor_SMD:R_0805_2012Metric_Pad1.15x1.40mm_HandSolder" V 8630 -850 50  0001 C CNN
 F 3 "~" H 8700 -850 50  0001 C CNN
 	1    8700 -850

Commit message: Added capacitor voltages, added bulk capacitors for battery power supply, changed crystal, added bypass capacitors for higher frequencies
Parts:
- added C42: 470n_35V, Capacitor_SMD:C_0805_2012Metric_Pad1.15x1.40mm_HandSolder, symbol Device:C
- added C43, C44, C45, C46, C47, C48: 100n, Capacitor_SMD:C_0805_2012Metric_Pad1.15x1.40mm_HandSolder, symbol Device:C
- added C49, C50: 680u_35V, Capacitor_THT:CP_Radial_D10.0mm_P5.00mm, symbol Device:CP1
- C1: value 2u2 -> 2u2_16V
- C10, C12, C30, C33, C35, C36: value 4.7u_60V -> 4u7_35V
- C11: value 4u7_50V -> 4u7_35V
- C13, C14, C15: value 220n -> 100n_16V
- C16: value 100n -> 100n_10V
- C17: value 10u -> 10u_5V
- C18: value 100n -> 100n_5V
- C19: value 15p -> 100n_6V3
- C21: value 15p -> 100n_10V
- C3: value 2u2 -> 220n_16V
- C4: value 2u2 -> 1u_6V3
- C40, C7, C8: value 2u2 -> 2u2_5V
- C41: value 2u2 -> 2u2_3V3
- C5: value 22n -> 22n_50V
- C6: value 2u2 -> 1u_10V
- C9: value 2u2 -> 2u2_30V
- D4: footprint (none) -> Diode_SMD:D_SOD-123F
- R23: footprint (none) -> Resistor_SMD:R_0805_2012Metric_Pad1.15x1.40mm_HandSolder
- U2: footprint (none) -> AgriESC:DRV8303
- Y1: value 8M -> 8M_15p_capacitance
Connections:
- wire segments 553 -> 585

Commit message: Updated footprints, added analog supply
Parts:
- added C51: 2u2_5V, Capacitor_SMD:C_0805_2012Metric_Pad1.15x1.40mm_HandSolder, symbol Device:C
- added C52: 2u2_3V3, Capacitor_SMD:C_0805_2012Metric_Pad1.15x1.40mm_HandSolder, symbol Device:C
- added U15: MCP1700-3302E_SOT23, Package_TO_SOT_SMD:SOT-23, symbol Regulator_Linear:MCP1700-3302E_SOT23
- C29: value 2u2 -> 100n
- C48: value 100n -> 2u2
- SW1: footprint (none) -> AgriESC:1825232-1
- U10, U12, U13, U5, U6, U9: footprint (none) -> AgriESC:FDMS7698
- U11, U8: footprint (none) -> AgriESC:MAX9920
- Y1: footprint (none) -> Crystal:Crystal_HC49-U_Vertical
Connections:
- net labels added: VAA
- wire segments 585 -> 595
Other:
- note added: "1825232-1"
- note added: "FC4STCBAF8.0-BAG200"

Commit message: Reset annotation
Parts:
- L1: footprint (none) -> Inductor_THT:L_Radial_D9.5mm_P5.00mm_Fastron_07HVP
- renumbered C10 to C1, C28 to C10, C34 to C11, C29 to C12, C43 to C13, C44 to C14, C45 to C15, C46 to C16, C22 to C17, C23 to C18, C26 to C19, C12 to C2, C27 to C20, C48 to C21, C37 to C22, C38 to C23, C39 to C24, C31 to C25, C47 to C26, C20 to C27, C24 to C28, C32 to C29, C30 to C3, C25 to C30, C13 to C31, C5 to C32, C14 to C33, C1 to C34, C3 to C35, C15 to C36, C19 to C37, C4 to C38, C21 to C39, C33 to C4, C6 to C40, C11 to C41, C7 to C43, C8 to C44, C18 to C45, C16 to C46, C9 to C47, C17 to C48, C40 to C49, C35 to C5, C41 to C50, C36 to C6, C49 to C7, C50 to C8, C2 to C9, J8 to J1, J12 to J10, J5 to J11, J2 to J12, J1 to J2, J6 to J3, J7 to J4, J9 to J5, J11 to J6, J4 to J7, J3 to J8, J10 to J9, R13 to R1, R14 to R10, R32 to R11, R37 to R12, R12 to R13, R30 to R14, R35 to R15, R38 to R16, R39 to R17, R40 to R18, R23 to R19, R31 to R2, R24 to R20, R9 to R21, R26 to R22, R27 to R23, R28 to R24, R20 to R25, R21 to R26, R1 to R27, R22 to R28, R15 to R29, R36 to R3, R2 to R30, R3 to R31, R4 to R32, R16 to R33, R17 to R34, R19 to R35, R5 to R36, R18 to R37, R6 to R38, R7 to R39, R10 to R4, R8 to R40, R25 to R5, R33 to R6, R11 to R7, R29 to R8, R34 to R9, U5 to U1, U7 to U10, U2 to U11, U4 to U12, U3 to U13, U9 to U2, U12 to U3, U6 to U4, U10 to U5, U13 to U6, U1 to U7, U11 to U9
Other:
- note added: "LHL08TB220K"
